Commit message: start

File: description/gazebo_control.xacro (robot description, xacro)
@@ -1,7 +1,4 @@
 <?xml version="1.0"?>
-<robot xmlns:xacro="http://www.ros.org/wiki/xacro">
-    <gazebo>
-        <?xml version="1.0"?>
-<robot xmlns:xacro="http://www.ros.org/wiki/xacro">
+ <robot xmlns:xacro="http://www.ros.org/wiki/xacro">
     <gazebo>
         <plugin name='diff_drive' filename='libgazebo_ros_diff_drive.so'>
@@ -23,4 +20,2 @@
     </gazebo>
 </robot>
-    </gazebo>
-</robot>

File: description/robot.urdf.xacro (robot description, xacro)
@@ -3,5 +3,4 @@
     <xacro:include filename="robot_core.xacro" />
     <xacro:include filename="colours.xacro" />
-    <xacro:include filename="inertial_macros.xacro" />
     <xacro:include filename="gazebo_control.xacro" />
 </robot>

File: description/robot_core.xacro (robot description, xacro)
@@ -23,7 +23,4 @@
         <material name="white"/>
     </collision>
-     <xacro:inertial_box mass="0.5" x="0.3" y="0.3" z="0.15">
-        <origin xyz="0.15 0 0.075" rpy="0 0 0"/>
-    </xacro:inertial_box>
 </link>
 <!-- LEFT WHEEL -->
@@ -47,7 +44,4 @@
         <material name="blue"/>
     </collision>
-    <xacro:inertial_cylinder mass="0.1" length="0.05" radius="0.05">
-        <origin xyz="0 0 0" rpy="0 0 0"/>
-    </xacro:inertial_cylinder>
 </link>
 <!-- RIGHT WHEEL -->
@@ -71,7 +65,4 @@
         <material name="blue"/>
     </collision>
-    <xacro:inertial_cylinder mass="0.1" length="0.05" radius="0.05">
-        <origin xyz="0 0 0" rpy="0 0 0"/>
-    </xacro:inertial_cylinder>
 </link>
 <!-- CASTER WHEEL -->
@@ -94,7 +85,4 @@
         <material name="black"/>
     </collision>
-    <xacro:inertial_sphere mass="0.1" radius="0.05">
-        <origin xyz="0 0 0" rpy="0 0 0"/>
-    </xacro:inertial_sphere>
 </link>
 </robot>
